File: simulations/EPD-Boost-Driver/epd-boost-driver/epd-boost-driver.kicad_sch (KiCad schematic)
At the start: 4 parts

Commit message: cr2032 and epd boost
Parts:
- C1: value 100uF -> 300uF
- R1: value 15 -> 18
- V1: value 2.85 -> 2.51
Other:
- moved on the sheet: C1, I1, R1, V1
